File: carte.brd (EAGLE design)
At the start: 84 x 85 mm, 14 parts, among them J1 MIC127-140-A01

Commit message: régulation du contenu du répertoire GIT
Connections:
- net N$5 renamed P8
Changed lines of the file:
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@@
 <wire x1="24.285" y1="39.715" x2="25.75" y2="38.25" width="0.254" layer="1"/>
 </signal>
-<signal name="N$5">
+<signal name="P8">
 <contactref element="CAPTEUR_ULTRASON" pad="2"/>
 <contactref element="J1" pad="27"/>

Commit message: régulation du contenu du répertoire GIT
Parts:
- removed J1: MIC127-140-A01, MIC127-140-A01:DONGGUAN_MIC127-140-A01
- added CONNECTEUR_CARTE: MIC127-140-A01, MIC127-140-A01:DONGGUAN_MIC127-140-A01
- moved CAPTEUR_INFRAROUGE_DROIT 14.5 mm to (51.0, 60.0), flipped to the bottom
- moved CAPTEUR_INFRAROUGE_GAUCHE 14.5 mm to (35.5, 60.0), flipped to the bottom
- moved CAPTEUR_ULTRASON 12.0 mm to (42.0, 60.0)
- moved INTERRUPTEUR 12.0 mm to (39.0, 5.00)
- moved MOTEUR_DROIT 12.0 mm to (47.0, 30.0)
- moved MOTEUR_GAUCHE 12.0 mm to (37.0, 30.0)
- moved PILES 12.0 mm to (42.0, 40.0)
- moved PILOTE_MOTEUR_DROIT 12.0 mm to (47.0, 35.0)
- moved PILOTE_MOTEUR_GAUCHE 12.0 mm to (37.0, 35.0)
- moved R1 12.0 mm to (39.8, 56.1)
- moved R2 12.0 mm to (47.2, 63.8)
- moved R3 11.8 mm to (55.0, 59.5)
- moved R5 11.8 mm to (28.0, 58.0)
Connections:
- net 3V: now also CONNECTEUR_CARTE.10, CONNECTEUR_CARTE.11, CONNECTEUR_CARTE.12, CONNECTEUR_CARTE.13, CONNECTEUR_CARTE.14, CONNECTEUR_CARTE.9; no longer J1.10, J1.11, J1.12, J1.13, J1.14, J1.9
- net GND: now also CONNECTEUR_CARTE.1, CONNECTEUR_CARTE.2, CONNECTEUR_CARTE.3, CONNECTEUR_CARTE.4, CONNECTEUR_CARTE.5, CONNECTEUR_CARTE.6, CONNECTEUR_CARTE.S1, CONNECTEUR_CARTE.S2; no longer INTERRUPTEUR.3, J1.1, J1.2, J1.3, J1.4, J1.5, J1.6, J1.S1, J1.S2
- net P0: now also CONNECTEUR_CARTE.36, CONNECTEUR_CARTE.37, CONNECTEUR_CARTE.38, CONNECTEUR_CARTE.39; no longer J1.36, J1.37, J1.38, J1.39
- net P1: now also CONNECTEUR_CARTE.28, CONNECTEUR_CARTE.29, CONNECTEUR_CARTE.30, CONNECTEUR_CARTE.31; no longer J1.28, J1.29, J1.30, J1.31
- net P13: now also CONNECTEUR_CARTE.18; no longer J1.18
- net P14: now also CONNECTEUR_CARTE.17; no longer J1.17
- net P15: now also CONNECTEUR_CARTE.16; no longer J1.16
- net P16: now also CONNECTEUR_CARTE.15; no longer J1.15
- net P2: now also CONNECTEUR_CARTE.19, CONNECTEUR_CARTE.20, CONNECTEUR_CARTE.21, CONNECTEUR_CARTE.22; no longer J1.19, J1.20, J1.21, J1.22
- net P8: now also CONNECTEUR_CARTE.27; no longer J1.27
Routing:
- net N$6: track 4.93 -> 11.8 mm
- net 3V: track 186.3 -> 191.8 mm
- net P0: track 18.8 -> 23.2 mm
- net P2: track 12.1 -> 15.8 mm
- net N$11: track 3.99 -> 6.32 mm
Other:
- board text removed: "/Users/pierr_paul/Downloads/lien URL GitHub.bmp"

Commit message: régulation du contenu du répertoire GIT
Parts:
- moved MOTEUR_DROIT 10.0 mm to (37.0, 30.0)
- moved MOTEUR_GAUCHE 10.0 mm to (47.0, 30.0)
Connections:
- net N$1: now also MOTEUR_DROIT.2; no longer MOTEUR_GAUCHE.2
- net N$2: now also MOTEUR_DROIT.1; no longer MOTEUR_GAUCHE.1
- net N$3: now also MOTEUR_GAUCHE.1; no longer MOTEUR_DROIT.1
- net N$4: now also MOTEUR_GAUCHE.2; no longer MOTEUR_DROIT.2
Changed lines of the file:
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@@
 <attribute name="VALUE" x="34" y="-5" size="1.27" layer="27" align="center"/>
 </element>
-<element name="MOTEUR_DROIT" library="pinhead" library_urn="urn:adsk.eagle:library:325" package="1X02" package3d_urn="urn:adsk.eagle:package:22435/2" value="" x="47" y="30" smashed="yes" rot="R180">
+<element name="MOTEUR_GAUCHE" library="pinhead" library_urn="urn:adsk.eagle:library:325" package="1X02" package3d_urn="urn:adsk.eagle:package:22435/2" value="" x="47" y="30" smashed="yes" rot="R180">
 <attribute name="NAME" x="49.6162" y="28.1712" size="1.27" layer="25" ratio="10" rot="R180"/>
 <attribute name="POPULARITY" value="98" x="-34.28" y="117.63" size="1.778" layer="27" rot="R180" display="off"/>
 <attribute name="VALUE" x="49.54" y="33.175" size="1.27" layer="27" rot="R180"/>
 </element>
-<element name="MOTEUR_GAUCHE" library="pinhead" library_urn="urn:adsk.eagle:library:325" package="1X02" package3d_urn="urn:adsk.eagle:package:22435/2" value="" x="37" y="30" smashed="yes" rot="R180">
+<element name="MOTEUR_DROIT" library="pinhead" library_urn="urn:adsk.eagle:library:325" package="1X02" package3d_urn="urn:adsk.eagle:package:22435/2" value="" x="37" y="30" smashed="yes" rot="R180">
 <attribute name="NAME" x="39.6162" y="28.1712" size="1.27" layer="25" ratio="10" rot="R180"/>
 <attribute name="POPULARITY" value="98" x="-27.77" y="117.63" size="1.778" layer="27" rot="R180" display="off"/>
@@
 <signals>
 <signal name="N$1">
-<contactref element="MOTEUR_GAUCHE" pad="2"/>
+<contactref element="MOTEUR_DROIT" pad="2"/>
 <contactref element="PILOTE_MOTEUR_GAUCHE" pad="2"/>
 <wire x1="36.75" y1="33.95" x2="36.75" y2="32.75" width="0.254" layer="1"/>
@@
 </signal>
 <signal name="N$2">
-<contactref element="MOTEUR_GAUCHE" pad="1"/>
+<contactref element="MOTEUR_DROIT" pad="1"/>
 <contactref element="PILOTE_MOTEUR_GAUCHE" pad="3"/>
 <wire x1="37.25" y1="33.95" x2="37.25" y2="32.75" width="0.254" layer="1"/>
@@
 <signal name="N$3">
 <contactref element="PILOTE_MOTEUR_DROIT" pad="3"/>
-<contactref element="MOTEUR_DROIT" pad="1"/>
+<contactref element="MOTEUR_GAUCHE" pad="1"/>
 <wire x1="47.25" y1="33.95" x2="47.25" y2="32.75" width="0.254" layer="1"/>
 <wire x1="48.27" y1="31.73" x2="48.27" y2="30" width="0.254" layer="1"/>
@@
 <signal name="N$4">
 <contactref element="PILOTE_MOTEUR_DROIT" pad="2"/>
-<contactref element="MOTEUR_DROIT" pad="2"/>
+<contactref element="MOTEUR_GAUCHE" pad="2"/>
 <wire x1="46.75" y1="33.95" x2="46.75" y2="32.75" width="0.254" layer="1"/>
 <wire x1="45.73" y1="31.73" x2="45.73" y2="30" width="0.254" layer="1"/>
