File: carte.sch (EAGLE design)
At the start: 14 parts, among them J1 MIC127-140-A01

Commit message: régulation du contenu du répertoire GIT
Connections:
- net N$5 renamed P8
Changed lines of the file:
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@@
 <segment>
 <pinref part="CAPTEUR_ULTRASON" gate="A" pin="3"/>
-<wire x1="73.66" y1="147.32" x2="73.66" y2="119.38" width="0.1524" layer="91"/>
+<wire x1="73.66" y1="147.32" x2="73.66" y2="106.68" width="0.1524" layer="91"/>
 <pinref part="J1" gate="G$1" pin="P1_4/AIN"/>
 <wire x1="48.26" y1="88.9" x2="48.26" y2="93.98" width="0.1524" layer="91"/>
@@
 <wire x1="55.88" y1="93.98" x2="53.34" y2="93.98" width="0.1524" layer="91"/>
 <junction x="53.34" y="93.98"/>
-<wire x1="48.26" y1="93.98" x2="48.26" y2="101.6" width="0.1524" layer="91"/>
+<wire x1="48.26" y1="93.98" x2="48.26" y2="106.68" width="0.1524" layer="91"/>
 <junction x="48.26" y="93.98"/>
-<wire x1="48.26" y1="101.6" x2="137.16" y2="101.6" width="0.1524" layer="91"/>
-<wire x1="137.16" y1="101.6" x2="137.16" y2="119.38" width="0.1524" layer="91"/>
-<wire x1="137.16" y1="119.38" x2="73.66" y2="119.38" width="0.1524" layer="91"/>
+<wire x1="48.26" y1="106.68" x2="73.66" y2="106.68" width="0.1524" layer="91"/>
 </segment>
 </net>
@@
 </segment>
 </net>
-<net name="N$5" class="0">
+<net name="P8" class="0">
 <segment>
 <pinref part="CAPTEUR_ULTRASON" gate="A" pin="2"/>
-<wire x1="71.12" y1="147.32" x2="71.12" y2="129.54" width="0.1524" layer="91"/>
-<wire x1="71.12" y1="129.54" x2="58.42" y2="129.54" width="0.1524" layer="91"/>
+<wire x1="71.12" y1="147.32" x2="71.12" y2="114.3" width="0.1524" layer="91"/>
+<wire x1="71.12" y1="114.3" x2="58.42" y2="114.3" width="0.1524" layer="91"/>
 <pinref part="J1" gate="G$1" pin="P8"/>
-<wire x1="58.42" y1="129.54" x2="58.42" y2="88.9" width="0.1524" layer="91"/>
+<wire x1="58.42" y1="114.3" x2="58.42" y2="88.9" width="0.1524" layer="91"/>
 </segment>
 </net>

Commit message: régulation du contenu du répertoire GIT
Parts:
- CAPTEUR_INFRAROUGE_DROIT, CAPTEUR_INFRAROUGE_GAUCHE: LCSC (none) -> C264269
- CONNECTEUR_CARTE: LCSC (none) -> C5154027
- INTERRUPTEUR: LCSC (none) -> C5274464
- PILOTE_MOTEUR_DROIT, PILOTE_MOTEUR_GAUCHE: LCSC (none) -> C39159
- R1, R3: LCSC (none) -> C25804
- R2, R5: LCSC (none) -> C22775
- renumbered J1 to CONNECTEUR_CARTE
Connections:
- net GND: no longer INTERRUPTEUR.NO

Commit message: régulation du contenu du répertoire GIT
Parts:
- R1, R2, R3, R5: POPULARITY 1KΩ -> (none)
Changed lines of the file:
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@@
 <part name="R5" library="rcl" library_urn="urn:adsk.eagle:library:334" deviceset="R-EU_" device="R0603" package3d_urn="urn:adsk.eagle:package:23555/3" value="100Ω">
 <attribute name="LCSC" value="C22775"/>
-<attribute name="POPULARITY" value="1KΩ"/>
+<attribute name="POPULARITY" value=""/>
 </part>
 <part name="R1" library="rcl" library_urn="urn:adsk.eagle:library:334" deviceset="R-EU_" device="R0603" package3d_urn="urn:adsk.eagle:package:23555/3" value="10KΩ">
 <attribute name="LCSC" value="C25804"/>
-<attribute name="POPULARITY" value="1KΩ"/>
+<attribute name="POPULARITY" value=""/>
 </part>
 <part name="R2" library="rcl" library_urn="urn:adsk.eagle:library:334" deviceset="R-EU_" device="R0603" package3d_urn="urn:adsk.eagle:package:23555/3" value="100Ω">
 <attribute name="LCSC" value="C22775"/>
-<attribute name="POPULARITY" value="1KΩ"/>
+<attribute name="POPULARITY" value=""/>
 </part>
 <part name="R3" library="rcl" library_urn="urn:adsk.eagle:library:334" deviceset="R-EU_" device="R0603" package3d_urn="urn:adsk.eagle:package:23555/3" value="10KΩ">
 <attribute name="LCSC" value="C25804"/>
-<attribute name="POPULARITY" value="1KΩ"/>
+<attribute name="POPULARITY" value=""/>
 </part>
 <part name="CONNECTEUR_CARTE" library="MIC127-140-A01" deviceset="MIC127-140-A01" device="">

Commit message: régulation du contenu du répertoire GIT
Connections:
- net N$1: now also MOTEUR_DROIT.2; no longer MOTEUR_GAUCHE.2
- net N$2: now also MOTEUR_DROIT.1; no longer MOTEUR_GAUCHE.1
- net N$3: now also MOTEUR_GAUCHE.1; no longer MOTEUR_DROIT.1
- net N$4: now also MOTEUR_GAUCHE.2; no longer MOTEUR_DROIT.2
Other:
- moved on the sheet: MOTEUR_DROIT, MOTEUR_GAUCHE
Changed lines of the file:
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@@
 <part name="CAPTEUR_ULTRASON" library="pinhead" library_urn="urn:adsk.eagle:library:325" deviceset="PINHD-1X4" device="" package3d_urn="urn:adsk.eagle:package:22407/2"/>
 <part name="PILES" library="pinhead" library_urn="urn:adsk.eagle:library:325" deviceset="PINHD-1X2" device="" package3d_urn="urn:adsk.eagle:package:22435/2"/>
+<part name="MOTEUR_DROIT" library="pinhead" library_urn="urn:adsk.eagle:library:325" deviceset="PINHD-1X2" device="" package3d_urn="urn:adsk.eagle:package:22435/2"/>
 <part name="MOTEUR_GAUCHE" library="pinhead" library_urn="urn:adsk.eagle:library:325" deviceset="PINHD-1X2" device="" package3d_urn="urn:adsk.eagle:package:22435/2"/>
-<part name="MOTEUR_DROIT" library="pinhead" library_urn="urn:adsk.eagle:library:325" deviceset="PINHD-1X2" device="" package3d_urn="urn:adsk.eagle:package:22435/2"/>
 <part name="INTERRUPTEUR" library="KH-SS12F17-G5" deviceset="KH-SS12F17-G5" device="">
 <attribute name="LCSC" value="C5274464"/>
@@
 <attribute name="VALUE" x="123.19" y="124.46" size="1.778" layer="96"/>
 </instance>
-<instance part="MOTEUR_GAUCHE" gate="G$1" x="-7.62" y="33.02" smashed="yes" rot="R180">
+<instance part="MOTEUR_DROIT" gate="G$1" x="-7.62" y="33.02" smashed="yes" rot="R180">
 <attribute name="NAME" x="-1.27" y="27.305" size="1.778" layer="95" rot="R180"/>
 <attribute name="VALUE" x="-1.27" y="38.1" size="1.778" layer="96" rot="R180"/>
 </instance>
-<instance part="MOTEUR_DROIT" gate="G$1" x="160.02" y="30.48" smashed="yes">
+<instance part="MOTEUR_GAUCHE" gate="G$1" x="160.02" y="30.48" smashed="yes">
 <attribute name="NAME" x="153.67" y="36.195" size="1.778" layer="95"/>
 <attribute name="VALUE" x="153.67" y="25.4" size="1.778" layer="96"/>
@@
 <net name="N$1" class="0">
 <segment>
-<pinref part="MOTEUR_GAUCHE" gate="G$1" pin="2"/>
+<pinref part="MOTEUR_DROIT" gate="G$1" pin="2"/>
 <pinref part="PILOTE_MOTEUR_GAUCHE" gate="G$1" pin="OUT1"/>
 <wire x1="-5.08" y1="33.02" x2="22.86" y2="33.02" width="0.1524" layer="91"/>
@@
 <net name="N$2" class="0">
 <segment>
-<pinref part="MOTEUR_GAUCHE" gate="G$1" pin="1"/>
+<pinref part="MOTEUR_DROIT" gate="G$1" pin="1"/>
 <pinref part="PILOTE_MOTEUR_GAUCHE" gate="G$1" pin="OUT2"/>
 <wire x1="-5.08" y1="30.48" x2="22.86" y2="30.48" width="0.1524" layer="91"/>
@@
 <segment>
 <pinref part="PILOTE_MOTEUR_DROIT" gate="G$1" pin="OUT2"/>
-<pinref part="MOTEUR_DROIT" gate="G$1" pin="1"/>
+<pinref part="MOTEUR_GAUCHE" gate="G$1" pin="1"/>
 <wire x1="121.92" y1="33.02" x2="157.48" y2="33.02" width="0.1524" layer="91"/>
 </segment>
@@
 <segment>
 <pinref part="PILOTE_MOTEUR_DROIT" gate="G$1" pin="OUT1"/>
-<pinref part="MOTEUR_DROIT" gate="G$1" pin="2"/>
+<pinref part="MOTEUR_GAUCHE" gate="G$1" pin="2"/>
 <wire x1="121.92" y1="30.48" x2="157.48" y2="30.48" width="0.1524" layer="91"/>
 </segment>
